File: MiniRadio/MiniRadio.kicad_sch (KiCad schematic)
At the start: 40 parts, among them J1 USB_C_Receptacle_USB2.0, J2 SMA, J3 54-00178, SW1 Freq_Tune, SW2 Volume_Tune, SW3 Reset, SW4 Boot, U1 ESP32-S3-WROOM-1, U2 Si4735-D60-GU, U6 EA_DOGS164-A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

Commit message: f
Parts:
- J1: footprint other_components:MOLEX_2171750001 -> USB-C_Receptacle:2171750001
- J2: footprint other_components:LINX_CONSMA002-SMD-G-T -> CONSMA002_SMD_G_T:LINX_CONSMA002-SMD-G-T
- J3: footprint 54-00178:TENSILITY_54-00178 -> TensilityAudioJack:TENSILITY_54-00178
- SW1, SW2: footprint Rotary_Encoder:RotaryEncoder_Bourns_Vertical_PEC12R-3xxxF-Nxxxx -> RotaryEncoders:PEC12R-4XXXF-NXXXX_BRN
- U1: footprint PCM_Espressif:ESP32-S3-WROOM-1 -> ESP32_S3_WROOM_1U_N4:XCVR_ESP32-S3-WROOM-1U-N4
- U3: footprint other_components:CONV_TPS62085RLTR -> TPS62086RLTR:RLT0007A
- U4: footprint other_components:SOT91P240X110-3N -> D1213A-01SO-7 Diode:D1213A01SO7
- U5: footprint other_components:QFN50P300X300X80-17N -> MAX98357AETE+T:QFN50P300X300X80-17N
