File: MiniRadio/MiniRadio.kicad_pcb (KiCad board)
At the start: 2 copper layers, 3.2 x 1.1 mm, 39 parts, among them J1 USB_C_Receptacle_USB2.0, J2 SMA, J3 54-00178, SW1 Freq_Tune, SW2 Volume_Tune, SW3 Reset, SW4 Boot, U1 ESP32-S3-WROOM-1, U2 Si4735-D60-GU, U6 EA_DOGS164-A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

Commit message: almost finishsed pcb layout
Parts:
- moved C21 45.5 mm to (150.0, 124.0), turned to 90 degrees
- moved SW1 44.1 mm to (174.0, 120.0), turned to -90 degrees
- moved C6 43.1 mm to (130.0, 114.0)
- moved R2 41.0 mm to (136.7, 121.0)
- moved R1 41.0 mm to (136.7, 117.0)
- moved R3 41.0 mm to (136.7, 125.1)
- moved C1 39.2 mm to (151.0, 119.0)
- moved C7 36.7 mm to (136.0, 114.0)
- moved U2 35.4 mm to (166.0, 124.0), turned to 180 degrees
- moved U4 28.6 mm to (173.1, 108.0), turned to 180 degrees
- moved C19 24.1 mm to (146.0, 97.0), turned to -90 degrees
- moved U5 21.9 mm to (181.8, 109.5)
- moved SW3 16.7 mm to (153.0, 68.0), turned to 180 degrees
- moved C15 14.9 mm to (160.2, 74.0), turned to 180 degrees
- moved C2 11.2 mm to (177.0, 83.0), turned to 90 degrees
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Routing:
- net +3.3V: track 0.00 -> 103.7 mm, vias 0 -> 4
- net /RST_LCD: track 0.00 -> 98.3 mm, vias 0 -> 2
- net Net-(U1-GPIO0/BOOT): track 0.00 -> 75.8 mm
- net /FMI: track 0.00 -> 75.7 mm, vias 0 -> 2
- net Net-(U2-DBYP): track 0.00 -> 73.3 mm, vias 0 -> 3
- net Net-(U1-EN): track 0.00 -> 63.5 mm, vias 0 -> 2
- net /USB_SUPPLY: track 0.00 -> 45.6 mm
- net /ROUT: track 0.00 -> 44.8 mm, vias 0 -> 2
- net +5V: track 0.00 -> 43.1 mm, vias 0 -> 2
- net /SCLK_LCD: track 0.00 -> 41.9 mm, vias 0 -> 2
- net /SDIO_LCD: track 0.00 -> 39.9 mm, vias 0 -> 2
- net /LOUT: track 0.00 -> 35.3 mm, vias 0 -> 2
- net /BATT_SUPPLY: track 0.00 -> 30.3 mm, vias 0 -> 4
- net /VOL_A: track 0.00 -> 29.5 mm, vias 0 -> 1
- net /VOL_B: track 0.00 -> 28.3 mm, vias 0 -> 1
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- added copper zone on B.Cu, net GND
- added copper zone on F.Cu, net GND
Other:
- board size 3.2 x 1.1 mm -> 77 x 72 mm
